File: zigbee_coordinator.kicad_pcb (KiCad board)
At the start: 2 copper layers, 33.5 x 33.5 mm, 51 parts, among them J1 USB_C_Receptacle_USB2.0, J2 Conn_01x01_Male, J3 Conn_01x01_Male, J4 Conn_01x01_Male, J5 Conn_01x01_Male, J6 Conn_01x01_Male, J7 Conn_01x01_Male, J8 Conn_01x01_Male, Q1 Q_PMOS_GSD, Q2 2N7002, U1 93LCxxBxxOT, U2 MCP1603-OS, U3 FT232H, U4 74LVC126, Y1 12MHz

Commit message: First alpha release
Parts:
- removed C15: 100n, Capacitor_SMD:C_0805_2012Metric
- removed C16: 10u, Capacitor_SMD:C_0805_2012Metric
- removed Q1: Q_PMOS_GSD, Inductor_SMD:L_0805_2012Metric
- removed Q2: 2N7002, Package_TO_SOT_SMD:SOT-23
- removed R12, R13: 12k, Resistor_SMD:R_0805_2012Metric
- removed R14, R15: 2k, Resistor_SMD:R_0805_2012Metric
- removed the Y1 at (186.6, 64.6)
- removed the Y1 at (195.6, 77.7)
- added D2: LED, LED_SMD:LED_0805_2012Metric, B.Cu at (122.2, 113.3)
- added F1: Polyfuse 150mA, Fuse:Fuse_0805_2012Metric, F.Cu at (122.7, 105.8)
- added J10: CONN_POGO, pogopin:pogopin, B.Cu at (121.2, 123.7)
- added J11: CONN_POGO, pogopin:pogopin, B.Cu at (121.2, 120.4)
- added J12: SWD_HOLES, pogopin:SWD_holes, F.Cu at (104.3, 100.0)
- added J13: UART_HOLES, pogopin:UART_holes, F.Cu at (111.5, 102.4)
- added J9: CONN_POGO, pogopin:pogopin, B.Cu at (93.6, 125.1)
- added U5: 74LVC126, Package_SO:TSSOP-14_4.4x5mm_P0.65mm, F.Cu at (99.4, 108.8)
- added U6: TPS22917DBV, Package_TO_SOT_SMD:SOT-23-6, F.Cu at (100.4, 118.6)
- added Y1: 12MHz, Crystal:Crystal_SMD_0603-2Pin_6.0x3.5mm, F.Cu at (115.6, 124.4)
- C10, C8: value 100n -> 27p
- C11: value 27p -> 10u
- C13, C3: value 100n -> 10u
- C7: value 10u -> 100n
- C9: value 27p -> 100n
- J2: value Conn_01x01_Male -> VCC_SEL; footprint pogopin:pogopin -> Connector_PinHeader_1.27mm:PinHeader_1x04_P1.27mm_Horizontal
- J3: value Conn_01x01_Male -> SWD_PADS; footprint pogopin:pogopin -> pogopin:SWD_pads
- J4: value Conn_01x01_Male -> UART_PADS; footprint pogopin:pogopin -> pogopin:UART_pads
- J5, J6, J7, J8: value Conn_01x01_Male -> CONN_POGO; moved to B.Cu
- L1: value 600R/0.5A -> 3.3uH
- L2: value 3.3uH -> 600R/0.5A
- R1: value 12k -> 5k1
- R11, R8: value 2k -> 12k
- R3: value 5k1 -> 12k
- R7: value 12k -> 2k
- moved R3 118.5 mm to (93.3, 115.8), turned to 180 degrees
- moved R4 115.7 mm to (93.3, 113.9), turned to 180 degrees
- moved R9 115.0 mm to (101.2, 114.4), turned to 270 degrees
- moved C1 112.0 mm to (93.3, 121.4), turned to 180 degrees
- moved R11 110.9 mm to (103.2, 118.8), turned to 90 degrees
- moved U1 108.3 mm to (93.3, 118.6)
- moved R6 106.8 mm to (111.1, 124.5), turned to 90 degrees
- moved R8 105.0 mm to (105.1, 106.4), turned to 90 degrees
- moved R10 104.1 mm to (103.2, 106.4), turned to 90 degrees
- moved C14 103.9 mm to (110.6, 127.3)
- moved C5 102.0 mm to (107.6, 106.4), turned to 90 degrees
- moved C2 101.8 mm to (107.2, 120.0), turned to 180 degrees
- moved C12 99.3 mm to (115.5, 108.6)
- moved C3 96.3 mm to (120.8, 105.8), turned to 270 degrees
- moved C9 96.2 mm to (110.6, 120.0)
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Connections:
- C10 pad 1: +3V3 -> Net-(C10-Pad1)
- C12 pad 1: Net-(C12-Pad1) -> +3V3
- C13 pad 1: Net-(C12-Pad1) -> Net-(C13-Pad1)
- C14 pad 1: +3V3 -> Net-(C14-Pad1)
- C3 pad 1: +3V3 -> /VBUS
- C9 pad 1: Net-(C9-Pad1) -> +3V3
- D1 pad 1: D+ -> D-
- D1 pad 2: D- -> D+
- J1 pad A4: Net-(C7-Pad1) -> Net-(F1-Pad1)
- J1 pad A9: Net-(C7-Pad1) -> Net-(F1-Pad1)
- J1 pad B4: Net-(C7-Pad1) -> Net-(F1-Pad1)
- J1 pad B9: Net-(C7-Pad1) -> Net-(F1-Pad1)
- J2 pad 1: /~RESET -> +3V3
- J3 pad 1: 3V3_OUT -> Net-(J12-Pad1)
- J4 pad 1: /SWDIO -> Net-(J13-Pad1)
- J5 pad 1: /SWDCK -> RESET_OUT
- J6 pad 1: GND -> VCC_CONN
- J7 pad 1: Net-(J7-Pad1) -> /SWDIO
- J8 pad 1: Net-(J8-Pad1) -> /SWDCK
- L1 pad 1: Net-(C12-Pad1) -> Net-(L1-Pad1)
- L2 pad 1: Net-(L2-Pad1) -> Net-(C11-Pad1)
- L3 pad 1: Net-(C15-Pad1) -> Net-(C13-Pad1)
- R1 pad 1: +3V3 -> GND
- R1 pad 2: Net-(R1-Pad2) -> Net-(J1-PadB5)
- R10 pad 1: /SWDIO_OE -> /SWD_EN
- R11 pad 1: /SWD_EN -> +3V3
- R11 pad 2: Net-(Q2-Pad1) -> /~SWD_EN
- R3 pad 1: GND -> +3V3
- R3 pad 2: Net-(J1-PadB5) -> Net-(R3-Pad2)
- R4 pad 2: Net-(R1-Pad2) -> Net-(R3-Pad2)
- R5 pad 1: +3V3 -> Net-(R5-Pad1)
- R5 pad 2: Net-(R5-Pad2) -> GND
- R6 pad 1: +3V3 -> /~SLEEP
- R6 pad 2: Net-(R6-Pad2) -> GND
- R7 pad 1: Net-(R7-Pad1) -> /SWD_EN
- R7 pad 2: GND -> Net-(D2-Pad2)
- R8 pad 1: /~PWREN -> /SWDIO_OE
- R8 pad 2: Net-(Q1-Pad1) -> GND
- R9 pad 1: +3V3 -> /RESET
- R9 pad 2: /~PWREN -> GND
- U1 pad 1: Net-(R1-Pad2) -> Net-(R3-Pad2)
- U1 pad 4: Net-(R5-Pad2) -> Net-(U1-Pad4)
- U1 pad 5: Net-(R6-Pad2) -> Net-(U1-Pad5)
- U2 pad 1: Net-(C7-Pad1) -> /VBUS
- U2 pad 3: Net-(C7-Pad1) -> /VBUS
- U2 pad 5: Net-(L2-Pad1) -> Net-(L1-Pad1)
- U3 pad 1: Net-(C9-Pad1) -> Net-(C8-Pad1)
- U3 pad 2: Net-(C11-Pad1) -> Net-(C10-Pad1)
- U3 pad 29: /~RESET -> /RESET
- U3 pad 3: Net-(C12-Pad1) -> Net-(C11-Pad1)
- U3 pad 32: /~PWREN -> /~SLEEP
- U3 pad 37: Net-(C8-Pad1) -> Net-(C7-Pad1)
- U3 pad 44: Net-(R5-Pad2) -> Net-(U1-Pad4)
- U3 pad 45: Net-(R6-Pad2) -> Net-(U1-Pad5)
- U3 pad 5: Net-(R7-Pad1) -> Net-(R5-Pad1)
- U3 pad 8: Net-(C15-Pad1) -> Net-(C13-Pad1)
- U4 pad 14: 3V3_OUT -> IO_VCC
Routing:
- net +3V3: track 0.00 -> 85.8 mm, vias 0 -> 2
- net GND: track 0.00 -> 54.9 mm, vias 0 -> 23
- net /SWD_EN: track 0.00 -> 48.9 mm, vias 0 -> 10
- net /TXD: track 0.00 -> 44.2 mm, vias 0 -> 1
- net /RxD: track 0.00 -> 37.1 mm, vias 0 -> 1
- net Net-(U1-Pad4): track 0.00 -> 26.7 mm, vias 0 -> 2
- net Net-(R4-Pad1): track 0.00 -> 26.2 mm, vias 0 -> 2
- net /~SLEEP: track 0.00 -> 25.3 mm, vias 0 -> 4
- net Net-(U1-Pad5): track 0.00 -> 23.4 mm, vias 0 -> 2
- net /RXD_TDI: track 0.00 -> 23.3 mm, vias 0 -> 3
- net IO_VCC: track 0.00 -> 22.2 mm, vias 0 -> 1
- net /TXD_TCK: track 0.00 -> 22.0 mm, vias 0 -> 3
- net /SWDCK: track 0.00 -> 21.9 mm, vias 0 -> 1
- net /~RTS~_TDO: track 0.00 -> 20.4 mm, vias 0 -> 2
- net Net-(C8-Pad1): track 0.00 -> 20.3 mm, vias 0 -> 2
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- removed copper zone on F.Cu, net GND
Other:
- outline, holes or cut-outs redrawn
- net class Default: trace_width 0.1524 -> 0.2
- net class Power: clearance 0.1524 -> 0.2; trace_width 0.25 -> 0.3; via_dia 0.8 -> 0.6; via_drill 0.5 -> 0.3

Commit message: Apply fizzo's fixes
Parts:
- U4, U5: value 74LVC126 -> 74LVC126A
Connections:
- J1 pad A8: Net-(J1-PadA8) -> (no net)
- J1 pad B8: Net-(J1-PadB8) -> (no net)
- U3 pad 16: /~CTS~_TMS -> (no net)
- U3 pad 17: Net-(U3-Pad17) -> (no net)
- U3 pad 18: Net-(U3-Pad18) -> (no net)
- U3 pad 19: Net-(U3-Pad19) -> (no net)
- U3 pad 20: Net-(U3-Pad20) -> (no net)
- U3 pad 21: Net-(U3-Pad21) -> (no net)
- U3 pad 27: Net-(U3-Pad27) -> (no net)
- U3 pad 28: Net-(U3-Pad28) -> (no net)
- U3 pad 30: Net-(U3-Pad30) -> (no net)
- U3 pad 31: Net-(U3-Pad31) -> (no net)
- U3 pad 33: Net-(U3-Pad33) -> (no net)
- U3 pad 42: Net-(U3-Pad42) -> (no net)
- U4 pad 1: /SWD_EN -> (no net)
- U4 pad 10: /~SWD_EN -> /SWD_EN
- U4 pad 11: /SWDCK -> /TXD
- U4 pad 13: /SWD_EN -> /~SWD_EN
- U4 pad 2: /SWDIO -> (no net)
- U4 pad 3: /~RTS~_TDO -> (no net)
- U4 pad 8: /TXD -> /SWDCK
- U5 pad 10: Net-(U5-Pad10) -> GND
- U5 pad 2: GND -> /SWDIO
- U5 pad 3: /~SWD_EN -> /~RTS~_TDO
- U5 pad 4: /RESET -> GND
- U5 pad 5: GND -> /SWD_EN
- U5 pad 6: RESET_OUT -> /~SWD_EN
- U5 pad 8: Net-(U5-Pad8) -> RESET_OUT
- U5 pad 9: Net-(U5-Pad9) -> /RESET
- U6 pad 4: Net-(U6-Pad4) -> (no net)
- U6 pad 5: Net-(U6-Pad5) -> (no net)
Routing:
- net RESET_OUT: track 12.4 -> 16.5 mm
- net /~RTS~_TDO: track 20.4 -> 16.3 mm
- net /~SWD_EN: track 19.7 -> 23.5 mm
- net /TXD: track 44.2 -> 47.2 mm
- net /SWD_EN: track 48.9 -> 46.2 mm
- net GND: track 54.9 -> 52.1 mm, vias 23 -> 24
- net /RESET: track 9.10 -> 11.7 mm
- net /SWDIO: track 19.8 -> 21.2 mm, vias 1 -> 2
- net +3V3: track 85.8 -> 86.3 mm
- net IO_VCC: track 22.2 -> 22.4 mm, vias 1 -> 0
