File: zigbee_coordinator.sch (KiCad schematic (older format))
At the start: 53 parts, among them J1 USB_C_Receptacle_USB2.0, J2 SERIAL_CONN, J3 POWER_SWD_CONN, Q1 Q_PMOS_GSD, U1 93LCxxB, U2 TPS22917DBV, U3 TPS562200, U4 FT232H, U5 74HC126, Y1 12MHz

Commit message: Before second 74LVC126
Parts:
- removed C1, C21, C9: 10u, symbol Device:C
- removed C16, C23, C3: 100n, symbol Device:C
- removed C4: 2.2nF, symbol Device:C
- removed D1, D2: D_TVS, symbol Device:D_TVS
- removed J2: SERIAL_CONN, symbol Connector:Conn_01x02_Male
- removed J3: POWER_SWD_CONN, symbol Connector:Conn_01x05_Male
- removed R14: 2k, symbol Device:R
- removed R8: 35k, symbol Device:R
- removed R9: 12k, symbol Device:R
- removed U1: 93LCxxB, symbol Memory_EEPROM:93LCxxB
- removed U2: TPS22917DBV, Package_TO_SOT_SMD:SOT-23-6, symbol Power_Management:TPS22917DBV
- removed U3: TPS562200, Package_TO_SOT_SMD:SOT-23-6, symbol Regulator_Switching:TPS562200
- added D1: D_TVS_x2_AAC, Package_TO_SOT_SMD:SOT-23, symbol Device:D_TVS_x2_AAC
- added F?: Polyfuse 150mA, symbol Device:Polyfuse
- added J2: SWD_POGO_PADS, symbol Connector:Conn_01x05_Female
- added J3: UART_POGO_PADS, symbol Connector:Conn_01x02_Female
- added J4: SWD_POGO, symbol Connector:Conn_01x05_Male
- added J5: SWD_CASTELLATED, symbol Connector:Conn_01x05_Female
- added J6: UART_CASTELLATED, symbol Connector:Conn_01x02_Female
- added J7: UART_POGO, symbol Connector:Conn_01x02_Male
- added J?: VCC_SEL, symbol Connector:Conn_01x04_Male
- added Q2: 2N7002, Package_TO_SOT_SMD:SOT-23, symbol Transistor_FET:2N7002
- added R13, R? (x2): 12k, Resistor_SMD:R_0805_2012Metric, symbol Device:R
- added U1: 93LCxxBxxOT, Package_TO_SOT_SMD:SOT-23-6, symbol Memory_EEPROM:93LCxxBxxOT
- added U2: MCP1603-OS, Package_TO_SOT_SMD:SOT-23-5, symbol mcp1603:MCP1603-OS
- C1: renamed from C2; footprint (none) -> Capacitor_SMD:C_0805_2012Metric
- C10: renamed from C14; footprint (none) -> Capacitor_SMD:C_0805_2012Metric
- C11: renamed from C15; footprint (none) -> Capacitor_SMD:C_0805_2012Metric
- C12: renamed from C17; footprint (none) -> Capacitor_SMD:C_0805_2012Metric
- C13: renamed from C18; footprint (none) -> Capacitor_SMD:C_0805_2012Metric
- C14: renamed from C19; footprint (none) -> Capacitor_SMD:C_0805_2012Metric
- C15: renamed from C20; footprint (none) -> Capacitor_SMD:C_0805_2012Metric
- C16: renamed from C22; footprint (none) -> Capacitor_SMD:C_0805_2012Metric
- C2: renamed from C5; footprint (none) -> Capacitor_SMD:C_0805_2012Metric
- C3: renamed from C6; footprint (none) -> Capacitor_SMD:C_0805_2012Metric
- C4: renamed from C8; footprint (none) -> Capacitor_SMD:C_0805_2012Metric
- C5: renamed from C10; footprint (none) -> Capacitor_SMD:C_0805_2012Metric
- C6: renamed from C11; footprint (none) -> Capacitor_SMD:C_0805_2012Metric
- C7: footprint (none) -> Capacitor_SMD:C_0805_2012Metric
- C8: renamed from C12; footprint (none) -> Capacitor_SMD:C_0805_2012Metric
- C9: renamed from C13; footprint (none) -> Capacitor_SMD:C_0805_2012Metric
- J1: footprint (none) -> Connector_USB:USB_C_Receptacle_GCT_USB4085
- L1, L3: value L -> 600R/0.5A; footprint (none) -> Inductor_SMD:L_0805_2012Metric
- L2, Q1: footprint (none) -> Inductor_SMD:L_0805_2012Metric
- R1: renamed from R3; footprint (none) -> Resistor_SMD:R_0805_2012Metric
- R10: renamed from R13; footprint (none) -> Resistor_SMD:R_0805_2012Metric
- R11: renamed from R15; footprint (none) -> Resistor_SMD:R_0805_2012Metric
- R12, R4, R5, R6, R7: footprint (none) -> Resistor_SMD:R_0805_2012Metric
- R2: renamed from R1; footprint (none) -> Resistor_SMD:R_0805_2012Metric
- R3: renamed from R2; footprint (none) -> Resistor_SMD:R_0805_2012Metric
- R8: renamed from R11; footprint (none) -> Resistor_SMD:R_0805_2012Metric
- R9: renamed from R10; footprint (none) -> Resistor_SMD:R_0805_2012Metric
- U3: renamed from U4; footprint (none) -> Package_QFP:LQFP-48_7x7mm_P0.5mm
- U4: renamed from U5; value 74HC126 -> 74LVC126; footprint (none) -> Package_SO:TSSOP-14_4.4x5mm_P0.65mm
- Y1: footprint (none) -> Crystal:Crystal_SMD_HC49-SD
Connections:
- net +3V3: now also C1.1, C10.1, C14.1, C2.1, C3.1, C4.1, C5.1, L2.2, R1.1, R5.1, R6.1, R8.1, U3.12 (VCCIO), U3.24 (VCCIO), U3.34 (~RESET), U3.40 (VREGIN), U3.46 (VCCIO), J?.4 (Pin_4), R13.1, U1.6 (VCC), U2.4 (VFB)
- net D+: now also D1.1 (A1)
- net D-: now also D1.2 (A2)
- net GND: now also D1.3 (common), J4.1 (Pin_1), Q2.2 (S), U1.2 (GND), U2.2 (GND); no longer U4.10 (4OE), U4.9 (4A)
- net RXD_TDI: now also R?.2
- net SWDCK: now also J4.2 (Pin_2)
- net SWDIO: now also J4.3 (Pin_3)
- net SWD_EN: now also R12.1
- net TXD_TCK: now also U4.9 (4A); no longer R12.2
- net ~PWREN: now also R8.2
- net ~RESET: now also J4.5 (Pin_5)
- net at R4.1, U3.43 (EEDATA): now also U1.3 (DI)
- net at R5.2, U3.44 (EECLK): now also U1.4 (CLK)
- net at R6.2, U3.45 (EECS): now also U1.5 (CS)
- net at L2.1: now also U2.5 (SW)
- net TXD: now reaches U4.8 (4Y)
- net TXD: now also R?.2
- net at Q1.1 (G), R9.2: no longer R8.2
- net at J1.A4 (VBUS), J1.A9 (VBUS), J1.B4 (VBUS)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: now also C7.1, U2.1 (VIN), U2.3 (~SHDN~)
- net at R1.2, R4.2: now also U1.1 (DO)
- removed net +3V0: C1.1, C10.1, C14.1, C4.1, C5.1, L2.2, Q1.2 (S), R1.1, R5.1, R6.1, R8.1, U3.12 (VCCIO), U3.24 (VCCIO), U3.34 (~RESET), U3.46 (VCCIO), U4.14 (VCC)
- net 3V0_OUT renamed IO_VCC
- net IO_VCC: now also U4.14 (VCC), F?.2
- net SWDIO_EN renamed SWDIO_OE
- removed net VBUS: C2.1, C3.1, C7.1, U3.40 (VREGIN)
- new net: J2.1 (Pin_1), J5.1 (Pin_1)
- new net: J2.2 (Pin_2), J5.2 (Pin_2)
- new net: J2.3 (Pin_3), J5.3 (Pin_3)
- new net: J2.4 (Pin_4), J5.4 (Pin_4)
- new net: J2.5 (Pin_5), J5.5 (Pin_5)
- new net: J7.2 (Pin_2), R?.1
- new net: J7.1 (Pin_1), R?.1
- new net: J3.1 (Pin_1), J6.1 (Pin_1)
- new net: J3.2 (Pin_2), J6.2 (Pin_2)
- new net: F?.1, J?.1 (Pin_1)
- new net: J?.3 (Pin_3), Q1.2 (S)
- new net: Q2.1 (G), R12.2
- new net VCC_CONN: J4.4 (Pin_4), J?.2 (Pin_2)
- new net ~SWD_EN: Q2.3 (D), R13.2, U4.10 (4OE)
- no-connect marks 15 -> 14
Other:
- note added: "Battery"
- note added: "Must be used in\nopen-drain mode"
- note added: "USB"
- note removed: "Place near\nVCCD"
- note removed: "Probably\nnot needed"
- note removed: "USB max inrush current is 100 mA\n2.2nF Cf = 4ms of rise time\nI=V*C/t=5V*25uF/4ms=31mA"
- note removed: "VCCD is a power output\nwhen VREGIN is at 5V"
- moved on the sheet: C1, C10, C11, C12, C13, C14, C15, C16, C2, C3, C4, C5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

Commit message: First alpha release
Parts:
- removed C13, C15, C3: 100n, Capacitor_SMD:C_0805_2012Metric, symbol Device:C
- removed J2: SWD_POGO_PADS, symbol Connector:Conn_01x05_Female
- removed J3: UART_POGO_PADS, symbol Connector:Conn_01x02_Female
- removed J4: SWD_POGO, symbol Connector:Conn_01x05_Male
- removed J7: UART_POGO, symbol Connector:Conn_01x02_Male
- removed Q1: Q_PMOS_GSD, Inductor_SMD:L_0805_2012Metric, symbol Device:Q_PMOS_GSD
- removed Q2: 2N7002, Package_TO_SOT_SMD:SOT-23, symbol Transistor_FET:2N7002
- removed R12, R9: 2k, Resistor_SMD:R_0805_2012Metric, symbol Device:R
- removed R5, R6, R? (x2): 12k, Resistor_SMD:R_0805_2012Metric, symbol Device:R
- added C14: 10u, Capacitor_SMD:C_0805_2012Metric, symbol Device:C
- added D2: LED, LED_SMD:LED_0805_2012Metric, symbol Device:LED
- added J10, J11, J5, J6, J7, J8, J9: CONN_POGO, pogopin:pogopin, symbol Connector:Conn_01x01_Male
- added J3: SWD_PADS, pogopin:SWD_pads, symbol Connector:Conn_01x05_Female
- added J4: UART_PADS, pogopin:UART_pads, symbol Connector:Conn_01x02_Female
- added R10: 12k, Resistor_SMD:R_0805_2012Metric, symbol Device:R
- added R7: 2k, Resistor_SMD:R_0805_2012Metric, symbol Device:R
- added U5: 74LVC126, Package_SO:TSSOP-14_4.4x5mm_P0.65mm, symbol 74hc126:74HC126
- added U6: TPS22917DBV, Package_TO_SOT_SMD:SOT-23-6, symbol Power_Management:TPS22917DBV
- F1: renamed from F?; footprint (none) -> Fuse:Fuse_0805_2012Metric
- J12: renamed from J5; value SWD_CASTELLATED -> SWD_HOLES; footprint (none) -> pogopin:SWD_holes
- J13: renamed from J6; value UART_CASTELLATED -> UART_HOLES; footprint (none) -> pogopin:UART_holes
- J2: renamed from J?; footprint (none) -> Connector_PinHeader_1.27mm:PinHeader_1x04_P1.27mm_Horizontal
- Y1: footprint Crystal:Crystal_SMD_HC49-SD -> Crystal:Crystal_SMD_0603-2Pin_6.0x3.5mm
- renumbered C11 to C10, C12 to C11, C14 to C12, C16 to C13, C7 to C3, C8 to C7, C9 to C8, C10 to C9, L2 to L1, L1 to L2, R2 to R1, R13 to R11, R3 to R2, R1 to R3, R7 to R5, R8 to R6, R10 to R8, R11 to R9
Connections:
- net +3V3: now also J2.1 (Pin_1), U5.14 (VCC); no longer J2.4 (Pin_4), R6.1
- net D+: now also D1.2 (A2); no longer D1.1 (A1)
- net D-: now also D1.1 (A1); no longer D1.2 (A2)
- net GND: now also R6.2, C14.2, D2.1 (K), J9.1 (Pin_1), R10.2, U5.2 (1A), U5.5 (2A), U5.7 (GND), U6.2 (GND)
- net IO_VCC: now also J2.4 (Pin_4), U6.6 (VOUT); no longer F1.2
- net RXD_TDI: now also U5.11 (3Y)
- net SWDCK: now also J8.1 (Pin_1)
- net SWDIO: now also J7.1 (Pin_1)
- net SWD_EN: now also R10.1, R7.1, U5.1 (1OE); no longer R9.1
- net TXD: now also J10.1 (Pin_1)
- net VCC_CONN: now also J2.3 (Pin_3), J6.1 (Pin_1); no longer J2.2 (Pin_2)
- net ~SWD_EN: now also U5.13 (3OE), U5.3 (1Y)
- net at J1.A4 (VBUS), J1.A9 (VBUS), J1.B4 (VBUS)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: now also F1.1; no longer C3.1, U2.1 (VIN), U2.3 (~SHDN~)
- net at J1.A5 (CC1): now also R2.2; no longer R1.2
- net at J1.B5 (CC2): now also R1.2; no longer R2.2
- net at J12.1 (Pin_1): now also J3.1 (Pin_1)
- net at J12.2 (Pin_2): now also J3.2 (Pin_2)
- net at J12.3 (Pin_3): now also J3.3 (Pin_3)
- net at J12.4 (Pin_4): now also J3.4 (Pin_4)
- net at J12.5 (Pin_5): now also J3.5 (Pin_5)
- net at J13.1 (Pin_1): now also J4.1 (Pin_1)
- net at J13.2 (Pin_2): now also J4.2 (Pin_2)
- net ~PWREN renamed ~SLEEP
- net ~SLEEP: now also R6.1, U6.3 (ON); no longer R6.2
- net ~RESET renamed RESET
- net RESET: now also R9.1, U5.4 (2OE)
- new net: C14.1, J2.2 (Pin_2), U6.1 (VIN)
- new net: D2.2 (A), R7.2
- new net RESET_OUT: J5.1 (Pin_1), U5.6 (2Y)
- new net RxD: J11.1 (Pin_1), U5.12 (3A)
- new net VBUS: C3.1, F1.2, U2.1 (VIN), U2.3 (~SHDN~)
- no-connect marks 14 -> 19
Other:
- note added: "Place near\n93LCxx VCC"
- note added: "Unused"
- note removed: "Must be used in\nopen-drain mode"
- moved on the sheet: C1, C10, C11, C12, C13, C2, C3, C4, C5, C6, C7, C8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

Commit message: Apply fizzo's fixes
Parts:
- removed U4, U5: 74LVC126, Package_SO:TSSOP-14_4.4x5mm_P0.65mm, symbol 74hc126:74HC126
- added U4, U5: 74LVC126A, Package_SO:TSSOP-14_4.4x5mm_P0.65mm, symbol 74lvc126:74LVC126A
Connections:
- net +3V3: now also U5.14 (VCC)
- net GND: now also U4.7 (GND), U5.10 (3OE), U5.4 (2OE), U5.7 (GND)
- net IO_VCC: now also U4.14 (VCC)
- net RESET: now also U5.9 (3A)
- net RESET_OUT: now also U5.8 (3Y)
- net RXD_TDI: now also U4.5 (2A), U5.11 (4Y)
- net RxD: now also U5.12 (4A)
- net SWDCK: now also U4.8 (3Y)
- net SWDIO: now also U4.6 (2Y), U5.2 (1A)
- net SWDIO_OE: now also U4.4 (2OE)
- net SWD_EN: now also U4.10 (3OE), U5.1 (1OE), U5.5 (2A)
- net TXD: now also U4.11 (4Y)
- net TXD_TCK: now also U4.12 (4A), U4.9 (3A)
- net ~RTS~_TDO: now also U5.3 (1Y)
- net ~SWD_EN: now also U4.13 (4OE), U5.13 (4OE), U5.6 (2Y)
Other:
- moved on the sheet: D2, J10, J11, R10, R11, R7, R8, R9

Commit message: Finalize
Other:
- moved on the sheet: J10, J11
Changed lines of the file:
@@
 	-1   0    0    -1
 $EndComp
-Text Label 14350 4150 0    50   ~ 0
+Text Label 14350 4050 0    50   ~ 0
 TXD
 Text Label 8150 4250 0    50   ~ 0
@@
 Entry Wire Line
 	9300 7100 9400 7200
-Text Label 14350 4250 0    50   ~ 0
+Text Label 14350 4150 0    50   ~ 0
 RxD
 Text Label 13650 5650 0    50   ~ 0
@@
 Wire Wire Line
 	10550 6250 10550 5650
-Text Notes 15950 6300 0    50   ~ 0
+Text Notes 13600 3200 0    50   ~ 0
 Unused
 Connection ~ 10150 5950
@@
 L Connector:Conn_01x01_Male J10
 U 1 1 5E3BAC00
+P 14800 4050
+F 0 "J10" H 14750 4050 50  0000 R CNN
+F 1 "CONN_POGO" H 14600 4050 50  0000 R CNN
+F 2 "pogopin:pogopin" H 14800 4050 50  0001 C CNN
+F 3 "~" H 14800 4050 50  0001 C CNN
+	1    14800 4050
+	-1   0    0    1
+$EndComp
+$Comp
+L Connector:Conn_01x01_Male J11
+U 1 1 5E3BAC0A
 P 14800 4150
-F 0 "J10" H 14750 4150 50  0000 R CNN
+F 0 "J11" H 14750 4150 50  0000 R CNN
 F 1 "CONN_POGO" H 14600 4150 50  0000 R CNN
 F 2 "pogopin:pogopin" H 14800 4150 50  0001 C CNN
 F 3 "~" H 14800 4150 50  0001 C CNN
 	1    14800 4150
-	-1   0    0    1
-$EndComp
-$Comp
-L Connector:Conn_01x01_Male J11
-U 1 1 5E3BAC0A
-P 14800 4250
-F 0 "J11" H 14750 4250 50  0000 R CNN
-F 1 "CONN_POGO" H 14600 4250 50  0000 R CNN
-F 2 "pogopin:pogopin" H 14800 4250 50  0001 C CNN
-F 3 "~" H 14800 4250 50  0001 C CNN
-	1    14800 4250
 	-1   0    0    1
 $EndComp
@@
 NoConn ~ 13500 3150
 Wire Wire Line
-	14100 4050 14100 4150
-Wire Wire Line
-	14100 4150 14600 4150
-Wire Wire Line
-	13500 4050 14100 4050
-Wire Wire Line
-	14600 4250 14100 4250
-Wire Wire Line
-	14100 4250 14100 4950
+	14600 4150 14100 4150
+Wire Wire Line
+	14100 4150 14100 4950
 Wire Wire Line
 	14100 4950 12000 4950
+Wire Wire Line
+	12000 4950 12000 6250
+Wire Notes Line
+	12500 3350 13950 3350
+Wire Notes Line
+	13950 3350 13950 3000
+Wire Notes Line
+	13950 3000 12500 3000
+Wire Notes Line
+	12500 3000 12500 3350
+Wire Wire Line
+	13500 4050 14600 4050
 Wire Bus Line
 	12150 2400 12150 5350
 Wire Bus Line
 	9300 2400 9300 7100
-Wire Wire Line
-	12000 4950 12000 6250
 $EndSCHEMATC
